File: SCH/nanoleaf/nanoleaf.kicad_pcb (KiCad board)
At the start: 2 copper layers, 161 x 140 mm, 36 parts, among them J1 Conn_01x03_Pin, J2 Conn_01x03_Pin, J3 Conn_01x03_Pin, J7 Conn_01x05_Pin, J8 USB_C_Receptacle_USB2.0, SW1 SW_Push, SW2 SW_Push, SW3 SW_DPDT_x2, SW4 SW_DPDT_x2, SW6 SW_DPDT_x2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

Commit message: esp-c3-supermini
Parts:
- removed C4, C5, C6, C7: 100nF, Capacitor_SMD:C_0201_0603Metric
- removed C8, C9: 10uF, Capacitor_SMD:C_Elec_3x5.4
- removed J7: Conn_01x05_Pin, Connector_PinHeader_2.54mm:PinHeader_1x06_P2.54mm_Vertical
- removed J8: USB_C_Receptacle_USB2.0, Connector_USB:USB_C_Receptacle_HRO_TYPE-C-31-M-12
- removed R1, R2: 5K1, Resistor_SMD:R_0603_1608Metric
- removed R3: 10K, Resistor_SMD:R_0603_1608Metric
- removed the SW1 at (141.9, 65.6)
- removed SW4: SW_DPDT_x2, Button_Switch_SMD:SW_DPDT_CK_JS202011JCQN
- removed U1: ESP32-C3-MINI-1, Espressif:ESP32-C3-MINI-1
- removed U4: AMS1117CD-3.3, Package_TO_SOT_SMD:TO-252-3_TabPin2
- added U5: ESP32-C3_SUPERMINI, Espressif:MODULE_ESP32-C3_SUPERMINI_1, F.Cu at (132.5, 64.7)
- C1, C2, C3: footprint Capacitor_SMD:C_0201_0603Metric -> Capacitor_SMD:C_0603_1608Metric
- D1: renamed from D7; value SK6812 -> WS2812B; footprint LED_SMD:LED_SK6812_PLCC4_5.0x5.0mm_P3.2mm -> LED_SMD:LED_WS2812B_PLCC4_5.0x5.0mm_P3.2mm
- D10, D9: value SK6812 -> WS2812B; footprint LED_SMD:LED_SK6812_PLCC4_5.0x5.0mm_P3.2mm -> LED_SMD:LED_WS2812B_PLCC4_5.0x5.0mm_P3.2mm
- D2: renamed from D1; value SK6812 -> WS2812B; footprint LED_SMD:LED_SK6812_PLCC4_5.0x5.0mm_P3.2mm -> LED_SMD:LED_WS2812B_PLCC4_5.0x5.0mm_P3.2mm
- D3: renamed from D6; value SK6812 -> WS2812B; footprint LED_SMD:LED_SK6812_PLCC4_5.0x5.0mm_P3.2mm -> LED_SMD:LED_WS2812B_PLCC4_5.0x5.0mm_P3.2mm
- D4: renamed from D5; value SK6812 -> WS2812B; footprint LED_SMD:LED_SK6812_PLCC4_5.0x5.0mm_P3.2mm -> LED_SMD:LED_WS2812B_PLCC4_5.0x5.0mm_P3.2mm
- D5: renamed from D8; value SK6812 -> WS2812B; footprint LED_SMD:LED_SK6812_PLCC4_5.0x5.0mm_P3.2mm -> LED_SMD:LED_WS2812B_PLCC4_5.0x5.0mm_P3.2mm
- D6: renamed from D2; value SK6812 -> WS2812B; footprint LED_SMD:LED_SK6812_PLCC4_5.0x5.0mm_P3.2mm -> LED_SMD:LED_WS2812B_PLCC4_5.0x5.0mm_P3.2mm
- D7: renamed from D3; value SK6812 -> WS2812B; footprint LED_SMD:LED_SK6812_PLCC4_5.0x5.0mm_P3.2mm -> LED_SMD:LED_WS2812B_PLCC4_5.0x5.0mm_P3.2mm
- D8: renamed from D4; value SK6812 -> WS2812B; footprint LED_SMD:LED_SK6812_PLCC4_5.0x5.0mm_P3.2mm -> LED_SMD:LED_WS2812B_PLCC4_5.0x5.0mm_P3.2mm
- J1, J2, J3: footprint Connector_JST:JST_GH_SM03B-GHS-TB_1x03-1MP_P1.25mm_Horizontal -> Connector_JST:JST_PH_B3B-PH-SM4-TB_1x03-1MP_P2.00mm_Vertical
- SW2: value SW_Push -> SW_DPDT_x2; footprint Button_Switch_SMD:SW_SPST_B3U-1000P -> Button_Switch_SMD:SW_DPDT_CK_JS202011JCQN
- moved SW2 69.1 mm to (144.8, 139.2), turned to 0 degrees
- moved SW3 45.5 mm to (167.6, 99.7), turned to -60 degrees
- moved J3 1.76 mm to (174.1, 96.0), turned to -60 degrees
- moved J2 1.43 mm to (144.5, 146.1), turned to 180 degrees
- moved J1 0.90 mm to (116.0, 96.1), turned to 60 degrees
- moved C3 0.76 mm to (144.7, 31.6)
- moved C1 0.52 mm to (135.6, 47.3)
- moved C2 0.52 mm to (135.6, 49.9)
- renumbered SW6 to SW1
Connections:
- D1 pad 1: GND -> +5V
- D1 pad 2: Net-(D6-DOUT) -> Net-(D1-DOUT)
- D1 pad 3: +5V -> GND
- D1 pad 4: Net-(D7-DOUT) -> Net-(D1-DIN)
- D10 pad 1: GND -> +5V
- D10 pad 2: Net-(D10-DIN) -> DOUT
- D10 pad 3: +5V -> GND
- D10 pad 4: DOUT -> Net-(D10-DIN)
- D2 pad 1: GND -> +5V
- D2 pad 2: DIN -> Net-(D2-DOUT)
- D2 pad 3: +5V -> GND
- D2 pad 4: Net-(D1-DOUT) -> DIN
- D3 pad 1: GND -> +5V
- D3 pad 2: Net-(D5-DOUT) -> Net-(D1-DIN)
- D3 pad 3: +5V -> GND
- D3 pad 4: Net-(D6-DOUT) -> Net-(D3-DIN)
- D4 pad 1: GND -> +5V
- D4 pad 2: Net-(D4-DOUT) -> Net-(D3-DIN)
- D4 pad 3: +5V -> GND
- D4 pad 4: Net-(D5-DOUT) -> Net-(D4-DIN)
- D5 pad 1: GND -> +5V
- D5 pad 2: Net-(D7-DOUT) -> Net-(D5-DOUT)
- D5 pad 3: +5V -> GND
- D5 pad 4: Net-(D8-DOUT) -> Net-(D1-DOUT)
- D6 pad 1: GND -> +5V
- D6 pad 2: Net-(D1-DOUT) -> Net-(D6-DOUT)
- D6 pad 3: +5V -> GND
- D7 pad 1: GND -> +5V
- D7 pad 2: Net-(D2-DOUT) -> Net-(D7-DOUT)
- D7 pad 3: +5V -> GND
- D7 pad 4: Net-(D3-DOUT) -> Net-(D6-DOUT)
- D8 pad 1: GND -> +5V
- D8 pad 2: Net-(D3-DOUT) -> Net-(D4-DIN)
- D8 pad 3: +5V -> GND
- D8 pad 4: Net-(D4-DOUT) -> Net-(D7-DOUT)
- D9 pad 1: GND -> +5V
- D9 pad 2: Net-(D8-DOUT) -> Net-(D10-DIN)
- D9 pad 3: +5V -> GND
- D9 pad 4: Net-(D10-DIN) -> Net-(D5-DOUT)
- J1 pad 3: GND -> Net-(J1-Pin_3)
- J2 pad 3: GND -> Net-(J2-Pin_3)
- J3 pad 3: GND -> Net-(J3-Pin_3)
- SW1 pad 1: DOUT -> GND
- SW1 pad 2: Net-(J1-Pin_1) -> Net-(J1-Pin_3)
- SW1 pad 4: (no net) -> DOUT
- SW1 pad 5: (no net) -> Net-(J1-Pin_1)
- SW1 pad 6: (no net) -> GND
- SW2 pad 2: EN -> Net-(J2-Pin_3)
- SW3 pad 1: DOUT -> GND
- SW3 pad 2: Net-(J2-Pin_1) -> Net-(J3-Pin_3)
- SW3 pad 4: (no net) -> DOUT
- SW3 pad 5: (no net) -> Net-(J3-Pin_1)
- SW3 pad 6: (no net) -> GND
Routing:
- net GND: track 117.3 -> 35.7 mm, vias 32 -> 19
- net +5V: track 441.6 -> 511.2 mm, vias 11 -> 7
- net +3V3: track 112.6 -> 43.4 mm, vias 2 -> 0
- net Net-(D3-DOUT): track 52.7 -> 0.00 mm
- net EN: track 42.9 -> 0.00 mm, vias 3 -> 0
- net Net-(D4-DIN): track 0.00 -> 42.3 mm
- net Net-(D3-DIN): track 0.00 -> 41.8 mm
- net Net-(D1-DIN): track 0.00 -> 41.2 mm
- net Net-(D8-DOUT): track 38.0 -> 0.00 mm
- net Net-(D4-DOUT): track 35.7 -> 0.00 mm
- net BOOT: track 31.5 -> 0.00 mm, vias 2 -> 0
- net D-: track 26.2 -> 0.00 mm, vias 2 -> 0
- net D+: track 24.2 -> 0.00 mm
- net DIN: track 163.5 -> 181.2 mm, vias 4 -> 2
- net ESP_RX: track 14.1 -> 0.00 mm
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- removed copper zone on F.Cu, net +3V3
Other:
- board text added: "DoubleULeaf_PCB v1 2023"
- board text removed: "BOOT"
- board text removed: "RST"

Commit message: switch and jst PH
Parts:
- J1, J2, J3: value Conn_01x03_Pin -> JST PH S3B PH SM4 TB; footprint Connector_JST:JST_PH_B3B-PH-SM4-TB_1x03-1MP_P2.00mm_Vertical -> Connector_JST:JST_PH_S3B-PH-SM4-TB_1x03-1MP_P2.00mm_Horizontal
- SW1, SW2, SW3: value SW_DPDT_x2 -> Mss22d18; footprint Button_Switch_SMD:SW_DPDT_CK_JS202011JCQN -> Button_Switch_SMD:SW_DPDT_CK_JS202011SCQN
- moved J2 7.46 mm to (138.9, 151.0), turned to 90 degrees
- moved J1 6.97 mm to (114.7, 89.3), turned to -30 degrees
- moved J3 6.67 mm to (180.3, 98.4), turned to -150 degrees
- moved SW2 1.40 mm to (144.7, 140.6), turned to 180 degrees
- moved SW1 1.35 mm to (121.2, 98.6), turned to 60 degrees
- moved SW3 1.17 mm to (168.5, 98.9), turned to 120 degrees
Connections:
- J1 pad 1: Net-(J1-Pin_1) -> GND
- J1 pad MP: (no net) -> GND
- J2 pad 1: Net-(J2-Pin_1) -> GND
- J2 pad MP: (no net) -> GND
- J3 pad 1: Net-(J3-Pin_1) -> GND
- J3 pad MP: (no net) -> GND
- SW1 pad 1: GND -> DIN
- SW1 pad 3: DIN -> DOUT
- SW1 pad 4: DOUT -> DIN
- SW1 pad 5: Net-(J1-Pin_1) -> Net-(J1-Pin_3)
- SW1 pad 6: GND -> DOUT
- SW2 pad 1: GND -> DIN
- SW2 pad 3: DIN -> DOUT
- SW2 pad 4: DOUT -> DIN
- SW2 pad 5: Net-(J2-Pin_1) -> Net-(J2-Pin_3)
- SW2 pad 6: GND -> DOUT
- SW3 pad 1: GND -> DIN
- SW3 pad 3: DIN -> DOUT
- SW3 pad 4: DOUT -> DIN
- SW3 pad 5: Net-(J3-Pin_1) -> Net-(J3-Pin_3)
- SW3 pad 6: GND -> DOUT
Routing:
- net +5V: track 511.2 -> 458.8 mm, vias 7 -> 2
- net Net-(J3-Pin_3): track 7.03 -> 19.2 mm
- net Net-(J1-Pin_3): track 8.45 -> 20.1 mm
- net Net-(D6-DOUT): track 44.4 -> 33.0 mm, vias 0 -> 2
- net Net-(D7-DOUT): track 45.0 -> 55.8 mm
- net Net-(J2-Pin_3): track 8.54 -> 19.2 mm
- net Net-(J3-Pin_1): track 8.95 -> 0.00 mm
- net Net-(D5-DOUT): track 43.4 -> 34.6 mm, vias 0 -> 2
- net DIN: track 181.2 -> 173.5 mm, vias 2 -> 4
- net DOUT: track 88.7 -> 96.0 mm
- net Net-(J1-Pin_1): track 6.06 -> 0.00 mm
- net Net-(J2-Pin_1): track 5.89 -> 0.00 mm
- net Net-(D1-DOUT): track 41.5 -> 37.8 mm
- net SDA: track 51.6 -> 50.6 mm
- net SCL: track 50.8 -> 49.9 mm
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